File: cad/pcb/reparaturhelfer/rev1-a/bluetooth.kicad_sch (KiCad schematic)
At the start: 62 parts, among them J201 Conn_01x02, J202 Conn_01x12, J203 Conn_01x08, J204 Conn_01x15, J205 Conn_01x05, J206 AudioJack3, J207 Conn_01x01, J208 Conn_01x01, J209 Conn_01x01, SW201 SW_Push, SW202 SW_Push, T201 1:1, T202 1:1, U201 1117 5.0V, U202 AD8656

Commit message: Add: Routing Bluetooth
Parts:
- removed H201, H202: MountingHole, MountingHole:MountingHole_3.2mm_M3, symbol Mechanical:MountingHole
- removed J203: Conn_01x08, Connector_PinHeader_2.54mm:PinHeader_1x08_P2.54mm_Vertical, symbol Connector_Generic:Conn_01x08
- added J204: Conn_01x07, Connector_PinHeader_2.54mm:PinHeader_1x07_P2.54mm_Vertical, symbol Connector_Generic:Conn_01x07
- FID201, FID202, FID203: footprint (none) -> Fiducial:Fiducial_1mm_Mask2mm
- H201: renamed from H203; footprint MountingHole:MountingHole_4.3mm_M4 -> MountingHole:MountingHole_3.2mm_M3
- H202: renamed from H204; footprint MountingHole:MountingHole_4.3mm_M4 -> MountingHole:MountingHole_3.2mm_M3
- H203: renamed from H205; footprint MountingHole:MountingHole_4.3mm_M4 -> MountingHole:MountingHole_3.2mm_M3
- H204: renamed from H206; footprint MountingHole:MountingHole_4.3mm_M4 -> MountingHole:MountingHole_3.2mm_M3
- RV201, RV202: footprint Potentiometer_SMD:Potentiometer_Vishay_TS53YL_Vertical -> Potentiometer_SMD:Potentiometer_Vishay_TS53YJ_Vertical; Bauteil Vishay TS53YL203MR10 -> 23A-20K
- renumbered J204 to J203
Connections:
- net +5VA is gone; now on net +5V: R202.2, R210.2
Other:
- moved on the sheet: SW201, SW202

Commit message: Add: PCB fertig
Parts:
- added R203, R204: 0, Resistor_SMD:R_0603_1608Metric, symbol Device:R
- renumbered R203 to R205, R204 to R206, R205 to R207, R206 to R208, R207 to R209, R208 to R210, R209 to R211, R210 to R212, R211 to R213, R212 to R214, R213 to R215, R214 to R216, R215 to R217, R216 to R218
Connections:
- net +5V: now also R203.1, R204.1, R204.2
- net +8V: now reaches C203.1, C204.1, C205.1, D201.1 (K), D202.1 (K), U201.3 (VI)
- net +8V: now also R203.2
Other:
- note added: "Alt. TL072 (8V)"
- moved on the sheet: C201, U202C
