File: cad/pcb/reparaturhelfer/rev1-a/power_supply.kicad_sch (KiCad schematic)
At the start: 43 parts, among them J301 Conn_01x01, J302 Conn_01x01, J303 Conn_01x01, J304 Conn_01x01, J305 Conn_01x01, J306 Conn_01x01, J307 Conn_01x01, J308 Conn_01x01, J309 Conn_01x01, J310 Conn_01x01, J311 Conn_01x01, J312 Conn_01x01, J313 Conn_01x01, J314 Conn_01x01, J315 Conn_01x01, J316 Conn_01x01, J317 Conn_01x01, J318 Conn_01x01, J319 Conn_01x01, J320 Conn_01x01, J321 Conn_01x01, J322 Conn_01x01, J323 Conn_01x01, J324 Conn_01x01, J325 Conn_01x01, J326 Conn_01x01

Commit message: Add: Routing Bluetooth
Parts:
- renumbered J326 to J317, J317 to J318, J318 to J319, J319 to J320, J320 to J321, J321 to J322, J322 to J323, J323 to J324, J324 to J325, J325 to J326
Changed lines of the file:
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@@
   (symbol (lib_id "Connector_Generic:Conn_01x01") (at 92.71 101.6 90) (mirror x) (unit 1)
     (in_bom yes) (on_board yes) (dnp no)
-    (property "Reference" "J318" (at 92.71 104.14 0)
+    (property "Reference" "J319" (at 92.71 104.14 0)
       (effects (font (size 1.27 1.27)) (justify left))
     )
@@
       (project "reparaturhelfer"
         (path "/93378ebd-f9ac-4734-8bdd-78f97f3ae344/b1ad4e02-2571-4f26-b0b3-3fc3a1bdaf53"
-          (reference "J318") (unit 1)
+          (reference "J319") (unit 1)
         )
       )
@@
   (symbol (lib_id "Connector_Generic:Conn_01x01") (at 166.37 101.6 90) (mirror x) (unit 1)
     (in_bom yes) (on_board yes) (dnp no)
-    (property "Reference" "J321" (at 166.37 104.14 0)
+    (property "Reference" "J322" (at 166.37 104.14 0)
       (effects (font (size 1.27 1.27)) (justify left))
     )
@@
       (project "reparaturhelfer"
         (path "/93378ebd-f9ac-4734-8bdd-78f97f3ae344/b1ad4e02-2571-4f26-b0b3-3fc3a1bdaf53"
-          (reference "J321") (unit 1)
+          (reference "J322") (unit 1)
         )
       )
@@
   (symbol (lib_id "Connector_Generic:Conn_01x01") (at 233.68 101.6 90) (mirror x) (unit 1)
     (in_bom yes) (on_board yes) (dnp no)
-    (property "Reference" "J323" (at 233.68 104.14 0)
+    (property "Reference" "J324" (at 233.68 104.14 0)
       (effects (font (size 1.27 1.27)) (justify left))
     )
@@
       (project "reparaturhelfer"
         (path "/93378ebd-f9ac-4734-8bdd-78f97f3ae344/b1ad4e02-2571-4f26-b0b3-3fc3a1bdaf53"
-          (reference "J323") (unit 1)
+          (reference "J324") (unit 1)
         )
       )
@@
   (symbol (lib_id "Connector_Generic:Conn_01x01") (at 240.03 101.6 90) (mirror x) (unit 1)
     (in_bom yes) (on_board yes) (dnp no)
-    (property "Reference" "J324" (at 240.03 104.14 0)
+    (property "Reference" "J325" (at 240.03 104.14 0)
       (effects (font (size 1.27 1.27)) (justify left))
     )
@@
       (project "reparaturhelfer"
         (path "/93378ebd-f9ac-4734-8bdd-78f97f3ae344/b1ad4e02-2571-4f26-b0b3-3fc3a1bdaf53"
-          (reference "J324") (unit 1)
+          (reference "J325") (unit 1)
         )
       )
@@
   (symbol (lib_id "Connector_Generic:Conn_01x01") (at 142.24 101.6 90) (mirror x) (unit 1)
     (in_bom yes) (on_board yes) (dnp no)
-    (property "Reference" "J320" (at 142.24 104.14 0)
+    (property "Reference" "J321" (at 142.24 104.14 0)
       (effects (font (size 1.27 1.27)) (justify left))
     )
@@
       (project "reparaturhelfer"
         (path "/93378ebd-f9ac-4734-8bdd-78f97f3ae344/b1ad4e02-2571-4f26-b0b3-3fc3a1bdaf53"
-          (reference "J320") (unit 1)
+          (reference "J321") (unit 1)
         )
       )
@@
   (symbol (lib_id "Connector_Generic:Conn_01x01") (at 264.16 101.6 90) (mirror x) (unit 1)
     (in_bom yes) (on_board yes) (dnp no)
-    (property "Reference" "J325" (at 264.16 104.14 0)
+    (property "Reference" "J326" (at 264.16 104.14 0)
       (effects (font (size 1.27 1.27)) (justify left))
     )
@@
       (project "reparaturhelfer"
         (path "/93378ebd-f9ac-4734-8bdd-78f97f3ae344/b1ad4e02-2571-4f26-b0b3-3fc3a1bdaf53"
-          (reference "J325") (unit 1)
+          (reference "J326") (unit 1)
         )
       )
@@
   (symbol (lib_id "Connector_Generic:Conn_01x01") (at 39.37 57.15 0) (mirror y) (unit 1)
     (in_bom yes) (on_board yes) (dnp no)
-    (property "Reference" "J326" (at 36.83 57.15 0)
+    (property "Reference" "J317" (at 36.83 57.15 0)
       (effects (font (size 1.27 1.27)) (justify left))
     )
@@
       (project "reparaturhelfer"
         (path "/93378ebd-f9ac-4734-8bdd-78f97f3ae344/b1ad4e02-2571-4f26-b0b3-3fc3a1bdaf53"
-          (reference "J326") (unit 1)
+          (reference "J317") (unit 1)
         )
       )
@@
   (symbol (lib_id "Connector_Generic:Conn_01x01") (at 39.37 81.28 0) (mirror y) (unit 1)
     (in_bom yes) (on_board yes) (dnp no)
-    (property "Reference" "J317" (at 36.83 81.28 0)
+    (property "Reference" "J318" (at 36.83 81.28 0)
       (effects (font (size 1.27 1.27)) (justify left))
     )
@@
       (project "reparaturhelfer"
         (path "/93378ebd-f9ac-4734-8bdd-78f97f3ae344/b1ad4e02-2571-4f26-b0b3-3fc3a1bdaf53"
-          (reference "J317") (unit 1)
+          (reference "J318") (unit 1)
         )
       )
@@
   (symbol (lib_id "Connector_Generic:Conn_01x01") (at 135.89 101.6 90) (mirror x) (unit 1)
     (in_bom yes) (on_board yes) (dnp no)
-    (property "Reference" "J319" (at 135.89 104.14 0)
+    (property "Reference" "J320" (at 135.89 104.14 0)
       (effects (font (size 1.27 1.27)) (justify left))
     )
@@
       (project "reparaturhelfer"
         (path "/93378ebd-f9ac-4734-8bdd-78f97f3ae344/b1ad4e02-2571-4f26-b0b3-3fc3a1bdaf53"
-          (reference "J319") (unit 1)
+          (reference "J320") (unit 1)
         )
       )
@@
   (symbol (lib_id "Connector_Generic:Conn_01x01") (at 190.5 101.6 90) (mirror x) (unit 1)
     (in_bom yes) (on_board yes) (dnp no)
-    (property "Reference" "J322" (at 190.5 104.14 0)
+    (property "Reference" "J323" (at 190.5 104.14 0)
       (effects (font (size 1.27 1.27)) (justify left))
     )
@@
       (project "reparaturhelfer"
         (path "/93378ebd-f9ac-4734-8bdd-78f97f3ae344/b1ad4e02-2571-4f26-b0b3-3fc3a1bdaf53"
-          (reference "J322") (unit 1)
-        )
-      )
+          (reference "J323") (unit 1)
+        )
+      )

Commit message: Add: PCB fertig
Parts:
- removed H301, H302, H303, H304, H305, H306, H307: MountingHole, MountingHole:MountingHole_4.3mm_M4, symbol Mechanical:MountingHole
- added H301, H302, H303, H304, H305, H306, H307: MountingHole_Pad, MountingHole:MountingHole_3.2mm_M3_Pad, symbol Mechanical:MountingHole_Pad
Connections:
- net gnd_a: now reaches C302.2, C303.2, C304.2, D303.2 (A), D304.2 (A), J319.1 (Pin_1), J320.1 (Pin_1), J321.1 (Pin_1), J322.1 (Pin_1)
- net gnd_a: now also H301.1, H302.1, H303.1, H305.1, H307.1
- net gnd_b: now reaches C305.2, C306.2, J323.1 (Pin_1), J324.1 (Pin_1), J325.1 (Pin_1), J326.1 (Pin_1)
- net gnd_b: now also H304.1, H306.1
