File: cad/pcb/reparaturhelfer/rev1-a/reparaturhelfer.kicad_pcb (KiCad board)
At the start: 2 copper layers, 99 x 99 mm, 165 parts, among them J201 Conn_01x02, J202 Conn_01x12, J203 Conn_01x15, J204 Conn_01x07, J205 Conn_01x05, J206 AudioJack3, J207 Conn_01x01, J208 Conn_01x01, J209 Conn_01x01, J301 Conn_01x01, J302 Conn_01x01, J303 Conn_01x01, J304 Conn_01x01, J305 Conn_01x01, J306 Conn_01x01, J307 Conn_01x01, J308 Conn_01x01, J309 Conn_01x01, J310 Conn_01x01, J311 Conn_01x01, J312 Conn_01x01, J313 Conn_01x01, J314 Conn_01x01, J315 Conn_01x01, J316 Conn_01x01, J317 Conn_01x01, J318 Conn_01x01, J319 Conn_01x01, J320 Conn_01x01, J321 Conn_01x01, J322 Conn_01x01, J323 Conn_01x01, J324 Conn_01x01, J325 Conn_01x01, J326 Conn_01x01, J401 Conn_01x01, J402 Conn_01x01, J403 Conn_01x01, J404 Conn_01x01, J405 Conn_01x01, J406 Conn_01x01, J407 Conn_01x01, J408 Conn_01x01, J409 Conn_01x01, J410 Conn_01x01, J411 Conn_01x01, J412 Conn_01x01, J413 Conn_01x01, J414 Conn_01x01, J415 Conn_01x01, J416 Conn_01x01, J417 Conn_01x01, J418 Conn_01x01, J419 Conn_01x01, J420 Conn_01x01, J421 Conn_01x01, J422 Conn_01x01, J423 Conn_01x01, J424 Conn_01x01, J425 Conn_01x01, J426 Conn_01x01, J427 Conn_01x01, J428 Conn_01x01, J429 Conn_01x01, J430 Conn_01x01, J431 Conn_01x01, J432 Conn_01x01, J433 Conn_01x01, J434 Conn_01x01, J435 Conn_01x01, J436 Conn_01x01, J501 Conn_01x03, SW201 SW_Push, SW202 SW_Push, T201 1:1, T202 1:1, U201 1117 5.0V, U202 AD8656

Commit message: Add: PCB fertig
Parts:
- added R203: 0, Resistor_SMD:R_0603_1608Metric, B.Cu at (95.2, 52.5)
- added R204: 0, Resistor_SMD:R_0603_1608Metric, B.Cu at (96.8, 52.5)
- C401, C403, C405, FID203: moved to B.Cu
- C412: footprint Capacitor_THT:C_Rect_L16.5mm_W7.0mm_P15.00mm_MKT -> Capacitor_THT:C_Rect_L7.0mm_W3.5mm_P2.50mm_P5.00mm
- H301, H302, H303, H304, H305, H306, H307: value MountingHole -> MountingHole_Pad; footprint MountingHole:MountingHole_4.3mm_M4 -> MountingHole:MountingHole_3.2mm_M3_Pad
- H501: footprint MountingHole:MountingHole_3mm_Pad -> MountingHole:MountingHole_3.2mm_M3_Pad
- H502: value MountingHole_Pad -> MountingHole; footprint MountingHole:MountingHole_3mm_Pad -> MountingHole:MountingHole_3.2mm_M3
- moved J305 359.9 mm to (171.8, 88.2)
- moved J316 355.5 mm to (175.5, 54.0)
- moved J314 355.5 mm to (168.0, 54.0)
- moved J307 351.5 mm to (163.0, 88.2)
- moved J315 351.4 mm to (171.8, 54.0)
- moved H306 351.1 mm to (175.8, 66.0)
- moved J326 349.9 mm to (175.5, 78.0), turned to 180 degrees
- moved J313 347.1 mm to (160.2, 54.0)
- moved J322 344.2 mm to (165.5, 107.0)
- moved J308 342.7 mm to (159.2, 88.2)
- moved H307 342.4 mm to (165.5, 97.5)
- moved J312 337.8 mm to (151.5, 54.0)
- moved J304 337.0 mm to (149.0, 88.2)
- moved J325 336.2 mm to (162.0, 78.0), turned to 180 degrees
- moved C306 330.4 mm to (163.9, 62.5), turned to -90 degrees
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- renumbered R203 to R205, R204 to R206, R205 to R207, R206 to R208, R207 to R209, R208 to R210, R209 to R211, R210 to R212, R211 to R213, R212 to R214, R213 to R215, R214 to R216, R215 to R217, R216 to R218
Connections:
- net Net-(D201-K) renamed +8V
- C302 pad 2: Net-(D303-A) -> /Power Supply/gnd_a
- C303 pad 2: Net-(D303-A) -> /Power Supply/gnd_a
- C304 pad 2: Net-(D303-A) -> /Power Supply/gnd_a
- C305 pad 2: Net-(J323-Pin_1) -> /Power Supply/gnd_b
- C306 pad 2: Net-(J323-Pin_1) -> /Power Supply/gnd_b
- C502 pad 2: Net-(J501-Pin_2) -> Net-(J501-Pin_3)
- C503 pad 1: Net-(J501-Pin_2) -> Net-(J501-Pin_3)
- D303 pad 2: Net-(D303-A) -> /Power Supply/gnd_a
- D304 pad 2: Net-(D303-A) -> /Power Supply/gnd_a
- J319 pad 1: Net-(D303-A) -> /Power Supply/gnd_a
- J320 pad 1: Net-(D303-A) -> /Power Supply/gnd_a
- J321 pad 1: Net-(D303-A) -> /Power Supply/gnd_a
- J322 pad 1: Net-(D303-A) -> /Power Supply/gnd_a
- J323 pad 1: Net-(J323-Pin_1) -> /Power Supply/gnd_b
- J324 pad 1: Net-(J323-Pin_1) -> /Power Supply/gnd_b
- J325 pad 1: Net-(J323-Pin_1) -> /Power Supply/gnd_b
- J326 pad 1: Net-(J323-Pin_1) -> /Power Supply/gnd_b
- J501 pad 2: Net-(J501-Pin_2) -> unconnected-(J501-Pin_2-Pad2)
- J501 pad 3: Earth -> Net-(J501-Pin_3)
Routing:
- net Net-(J303-Pin_1): track 0.00 -> 54.6 mm
- net Net-(D301-K): track 0.00 -> 52.7 mm
- net +8V: track 28.0 -> 72.1 mm, vias 1 -> 3
- net Net-(J311-Pin_1): track 0.00 -> 33.0 mm
- net Net-(D302-A): track 0.00 -> 23.7 mm
- net Net-(D301-A): track 0.00 -> 23.6 mm
- net Net-(J501-Pin_3): track 0.00 -> 21.2 mm
- net Net-(J315-Pin_1): track 0.00 -> 15.5 mm
- net Earth: track 9.99 -> 24.2 mm
- net Net-(J307-Pin_1): track 0.00 -> 12.1 mm
- net /Power Supply/gnd_a: track 0.00 -> 11.3 mm
- net Net-(J501-Pin_1): track 0.00 -> 11.1 mm
- net Net-(J427-Pin_1): track 0.00 -> 11.0 mm
- net Net-(J433-Pin_1): track 0.00 -> 10.2 mm
- net Net-(J434-Pin_1): track 0.00 -> 5.25 mm
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- added copper zone on B.Cu, net /Power Supply/gnd_a
- added copper zone on B.Cu, net /Power Supply/gnd_b
Other:
- board size 99 x 99 mm -> 99.5 x 99.5 mm
- board text added: "+"
- board text added: "Bluetooth Rev1-a 2024-01 Martin Wagner DL2WAG"
- board text added: "R 35mm"
- board text added: "R 60mm"
- board text added: "R 80mm"
- board text added: "erster Filter"
- board text added: "l"
- board text added: "links / mono"
- board text added: "r"
- board text added: "rechts"
- board text added: "zweiter Filter"
- board text added: "~"
